File: 555-gerador-PWM-r01.kicad_pcb (KiCad board)
At the start: 2 copper layers, 49.5 x 49.3 mm, 12 parts, among them J1 Saída PWM, J2 Alimentação, U1 NE555

Commit message: revisados furos (removido GND)
Routing:
- net GND: vias 4 -> 0
- net (no net): vias 0 -> 4
Changed lines of the file:
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@@
   )
   (setup
-    (last_trace_width 1)
+    (last_trace_width 0.25)
     (user_trace_width 0.4)
     (user_trace_width 0.6)
@@
       (padsonsilk false)
       (subtractmaskfromsilk false)
-      (outputformat 5)
+      (outputformat 1)
       (mirror false)
       (drillshape 0)
       (scaleselection 1)
-      (outputdirectory "svg-pwm-555/"))
+      (outputdirectory "Production-files-pwm-555-r01/"))
   )
   (net 0 "")
@@
   (segment (start 155.956 90.424) (end 155.956 88.30268) (width 1) (layer B.Cu) (net 9))
   (segment (start 155.956 88.30268) (end 154.77532 87.122) (width 1) (layer B.Cu) (net 9))
-  (via (at 118.872 130.556) (size 3.5) (drill 3.3) (layers F.Cu B.Cu) (net 9))
-  (via (at 162.814 130.556) (size 3.5) (drill 3.3) (layers F.Cu B.Cu) (net 9))
-  (via (at 162.814 86.868) (size 3.5) (drill 3.3) (layers F.Cu B.Cu) (net 9))
-  (via (at 118.872 86.868) (size 3.5) (drill 3.3) (layers F.Cu B.Cu) (net 9))
+  (via (at 118.872 130.556) (size 3.5) (drill 3.3) (layers F.Cu B.Cu) (net 0))
+  (via (at 162.814 130.556) (size 3.5) (drill 3.3) (layers F.Cu B.Cu) (net 0))
+  (via (at 162.814 86.868) (size 3.5) (drill 3.3) (layers F.Cu B.Cu) (net 0))
+  (via (at 118.872 86.868) (size 3.5) (drill 3.3) (layers F.Cu B.Cu) (net 0))
   (segment (start 142.24 115.062) (end 144.78 112.522) (width 1) (layer B.Cu) (net 10))
   (segment (start 142.24 116.332) (end 142.24 115.062) (width 1) (layer B.Cu) (net 10))
